Commit message: Add files via upload

File: usv_worlds/worlds/simple_obstacles.xacro (robot description, xacro)
@@ -9,8 +9,14 @@
     <xacro:simple_box name="box_east" x="25" y="-40" X="150" />
     <xacro:simple_box name="box_west" x="-10" y="160" X="80" />
-    <xacro:simple_box name="jetty_one" x="-17.5" y="7" z="0.50" X="65" Y="3" Z="1.0" color="Wood" />
+    <!--  Boxes to do static avoidance -->
+    <xacro:simple_box name="box_test" x="30" y="30" X="1" Y="1" Z="1" />
+    <xacro:simple_box name="box_test_two" x="15" y="15" X="2" Y="2" Z="1" />
+    <xacro:simple_box name="box_test_three" x="25" y="25" X="9" Y="9" Z="1" />
+    <!-- <xacro:simple_box name="box_test_four" x="19" y="18" X="2" Y="2" Z="1" /> -->
+    <!-- <xacro:simple_box name="box_test_five" x="20" y="10" X="2" Y="2" Z="1" /> -->
+  </xacro:macro>
+</world>
+    <!--<xacro:simple_box name="jetty_one" x="-17.5" y="7" z="0.50" X="65" Y="3" Z="1.0" color="Wood" />
     <xacro:simple_box name="jetty_two" x="-7.5" y="64" z="0.50" X="85" Y="4" Z="1.0" color="Wood" />
     <xacro:simple_box name="jetty_three" x="92.5" y="74" z="0.50" X="5" Y="112" Z="1.0" color="Wood" />
-    <xacro:simple_box name="box_north2" x="10" y="-20" Y="100" yaw="-1.0" />
-  </xacro:macro>
-</world>
+    <xacro:simple_box name="box_north2" x="10" y="-20" Y="100" yaw="-1.0" /> -->
