Commit message: Add files via upload

File: usv_worlds/worlds/Obstacle_Path.xacro (robot description, xacro)
@@ -4,5 +4,5 @@
   <!-- Load definition of simple_box -->
   <xacro:include filename="$(find usv_worlds)/worlds/simple_box.xacro" />
-  <xacro:macro name="Obstacle_path">
+  <xacro:macro name="Obstacle_Path">
     <!--  Boxes to do static avoidance -->
     <xacro:simple_box name="box_1" x="20" y="10" X="42" Y="2" Z="2" />
@@ -10,6 +10,11 @@
     <xacro:simple_box name="box_3" x="40" y="30" X="2" Y="40" Z="2" />
     <xacro:simple_box name="box_4" x="60" y="10" X="2" Y="40" Z="2" />
-    <xacro:simple_box name="box_5" x="80" y="50" X="82" Y="2" Z="1" />
-    <xacro:simple_box name="box_6" x="80" y="30" X="42" Y="2" Z="1" />
+    <xacro:simple_box name="box_5" x="75" y="50" X="72" Y="2" Z="1" />
+    <xacro:simple_box name="box_6" x="85" y="30" X="52" Y="2" Z="1" />
+    <!-- borders of the whole box-->
+    <xacro:simple_box name="box_north" x="111" y="20" Y="62" />
+    <xacro:simple_box name="box_south" x="-1" y="20" Y="62" />
+    <xacro:simple_box name="box_east" x="55" y="-11" X="112" />
+    <xacro:simple_box name="box_west" x="55" y="51" X="112" />
   </xacro:macro>
 </world>

File: usv_worlds/worlds/simple_box.xacro (robot description, xacro)
@@ -2,5 +2,5 @@
 <!-- Macro to insert simple obstacles into the world -->
 <world xmlns:xacro="http://ros.org/wiki/xacro">
-  <xacro:macro name="simple_box" params="name x:=0 y:=0 z:=1 roll:=0 pitch:=0 yaw:=0 X:=0.2 Y:=0.2 Z:=2 color:=DarkGray">
+  <xacro:macro name="simple_box" params="name x:=0 y:=0 z:=0 roll:=0 pitch:=0 yaw:=0 X:=0.2 Y:=0.2 Z:=2 color:=DarkGray">
     <model name='${name}'>
       <pose frame=''>${x} ${y} ${z} ${roll} ${pitch} ${yaw}</pose>

File: usv_worlds/worlds/simple_obstacles.xacro (robot description, xacro)
@@ -10,9 +10,8 @@
     <xacro:simple_box name="box_west" x="-10" y="160" X="80" />
     <!--  Boxes to do static avoidance -->
-    <xacro:simple_box name="box_test" x="30" y="30" X="1" Y="1" Z="1" />
-    <xacro:simple_box name="box_test_two" x="15" y="15" X="2" Y="2" Z="1" />
-    <xacro:simple_box name="box_test_three" x="25" y="25" X="9" Y="9" Z="1" />
-    <!-- <xacro:simple_box name="box_test_four" x="19" y="18" X="2" Y="2" Z="1" /> -->
-    <!-- <xacro:simple_box name="box_test_five" x="20" y="10" X="2" Y="2" Z="1" /> -->
+    <xacro:simple_box name="box_test" x="30" y="30" X="1" Y="1" Z="2" />
+    <xacro:simple_box name="box_test_two" x="15" y="15" X="2" Y="2" Z="2" />
+    <xacro:simple_box name="box_test_three" x="25" y="25" X="20" Y="20" Z="2" />
+    <xacro:simple_box name="box_test_four" x="23" y="20" X="20" Y="20" Z="2" />
   </xacro:macro>
 </world>

File: usv_worlds/worlds/usv.world.xacro (robot description, xacro)
@@ -35,6 +35,10 @@
       <uri>model://ocean</uri>
     </include>
-    <xacro:include filename="$(find usv_worlds)/worlds/simple_obstacles.xacro" />
-    <xacro:simple_obstacles />
+    <!-- Some simple obstacles in the way-->
+    <!--<xacro:include filename="$(find usv_worlds)/worlds/simple_obstacles.xacro" />
+    <xacro:simple_obstacles /> -->
+    <!-- simple trajectory to navigate between walls-->
+    <xacro:include filename="$(find usv_worlds)/worlds/Obstacle_Path.xacro" />
+    <xacro:Obstacle_Path />
   </world>
 </sdf>
