Commit message: Add files via upload

File: otter_gazebo/urdf/dynamics/otter_gazebo_dynamics_plugin.xacro (robot description, xacro)
@@ -34,5 +34,5 @@
         <wave_period0>5</wave_period0>
         <wave_direction0>-1 0</wave_direction0>
-        <wave_amp1>0.01</wave_amp1>
+        <wave_amp1>0.1</wave_amp1>
         <wave_period1>0.7</wave_period1>
         <wave_direction1>-0.7 0.7</wave_direction1>

File: otter_gazebo/urdf/dynamics/otter_gazebo_wind_plugin.xacro (robot description, xacro)
@@ -7,5 +7,5 @@
         <bodyName>base_link</bodyName>
         <!-- Wind -->
-        <wind_velocity_vector>0 0 0 </wind_velocity_vector>
+        <wind_velocity_vector>0 0 0 </wind_velocity_vector> <!--can change this to enable wind-->
         <wind_coeff_vector>0.5 0.5 0.33 </wind_coeff_vector>
       </plugin>

File: otter_gazebo/urdf/otter_gazebo.urdf.xacro (robot description, xacro)
@@ -61,5 +61,5 @@
   <!-- Add planar LIDAR -->
   <xacro:if value="$(arg lidar_enabled)">
-    <xacro:otter_lidar name="lidar" x="0" y="0.0" z="0.40" min_range="1.2" max_range="25" visualize="false" />
+    <xacro:otter_lidar name="lidar" x="0" y="0.0" z="0.40" min_range="1.2" max_range="25" visualize="false" /> <!--changed from 25 to 15 for testing 28/04-->
   </xacro:if>
   <!-- Add P3D ground truth -->

File: otter_gazebo/urdf/sensors/otter_lidar.xacro (robot description, xacro)
@@ -3,5 +3,5 @@
   <xacro:macro name="otter_lidar" params="name x:=0.5 y:=0 z:=0 R:=0 P:=0 Y:=0 min_range:=0.2 max_range:=25 visualize:=false">
     <link name="${name}_link">
-      <visual name="${name}_visual">>
+      <visual name="${name}_visual">
         <origin xyz="0 0 -0.05"/>
         <geometry>
@@ -25,5 +25,5 @@
           <scan>
             <horizontal>
-              <samples>720</samples>
+              <samples>2000</samples> <!--change from 720 to 2000-->
               <resolution>1</resolution>
               <min_angle>-3.14159265359</min_angle>
@@ -37,5 +37,5 @@
             <max>${max_range}</max>
             <!-- Linear resolution of the beam -->
-            <resolution>0.02</resolution>
+            <resolution>0.03</resolution> <!--changed from 0.02 to 0.03-->
           </range>
         </ray>

File: usv_worlds/worlds/Obstacle_Path.xacro (robot description, xacro)
@@ -6,15 +6,15 @@
   <xacro:macro name="Obstacle_Path">
     <!--  Boxes to do static avoidance -->
-    <xacro:simple_box name="box_1" x="20" y="10" X="42" Y="2" Z="2" />
+   <!--> <xacro:simple_box name="box_1" x="22" y="10" X="42" Y="2" Z="2" />
     <xacro:simple_box name="box_2" x="30" y="-10" X="62" Y="2" Z="2" />
     <xacro:simple_box name="box_3" x="40" y="30" X="2" Y="40" Z="2" />
     <xacro:simple_box name="box_4" x="60" y="10" X="2" Y="40" Z="2" />
     <xacro:simple_box name="box_5" x="75" y="50" X="72" Y="2" Z="1" />
-    <xacro:simple_box name="box_6" x="85" y="30" X="52" Y="2" Z="1" />
+    <xacro:simple_box name="box_6" x="85" y="30" X="52" Y="2" Z="1" />-->
     <!-- borders of the whole box-->
-    <xacro:simple_box name="box_north" x="111" y="20" Y="62" />
-    <xacro:simple_box name="box_south" x="-1" y="20" Y="62" />
-    <xacro:simple_box name="box_east" x="55" y="-11" X="112" />
-    <xacro:simple_box name="box_west" x="55" y="51" X="112" />
+    <xacro:simple_box name="box_north" x="111" y="0" Y="62" />
+    <xacro:simple_box name="box_south" x="-1" y="0" Y="62" />
+    <xacro:simple_box name="box_east" x="55" y="-24" X="112" />
+    <xacro:simple_box name="box_west" x="55" y="24" X="112" />
   </xacro:macro>
 </world>
@@ -22,3 +22,3 @@
     <xacro:simple_box name="jetty_two" x="-7.5" y="64" z="0.50" X="85" Y="4" Z="1.0" color="Wood" />
     <xacro:simple_box name="jetty_three" x="92.5" y="74" z="0.50" X="5" Y="112" Z="1.0" color="Wood" />
-    <xacro:simple_box name="box_north2" x="10" y="-20" Y="100" yaw="-1.0" /> -->
+    <xacro:simple_box name="box_north2" x="10" y="-22" Y="100" yaw="-1.0" /> -->

File: usv_worlds/worlds/moving_box.xacro (robot description, xacro)
@@ -3,6 +3,6 @@
 <sdf version="1.6">
    <world xmlns:xacro="http://ros.org/wiki/xacro">
-      <xacro:macro name="moving_box" params="name x:=0 y:=0 z:=1">
-        <actor name="${name}">
+      <xacro:macro name="moving_box" params="name x:=0 y:=0 z:=2">
+        <actor name="animated_box">
           <link name="box_link">
             <visual name="visual">
@@ -20,21 +20,21 @@
               <waypoint>
                   <time>0.0</time>
-                  <pose>${x}-1 ${y}-1 1 0 0 0</pose>
+                  <pose>-1 -1 1 0 0 0</pose>
               </waypoint>
               <waypoint>
                   <time>1.0</time>
-                  <pose>${x}-1 ${y}+1 1 0 0 0</pose>
+                  <pose>-1 1 1 0 0 0</pose>
               </waypoint>
               <waypoint>
                   <time>2.0</time>
-                  <pose>${x}+1 ${y}+1 1 0 0 0</pose>
+                  <pose>1 1 1 0 0 0</pose>
               </waypoint>
               <waypoint>
                   <time>3.0</time>
-                  <pose>${x}+1 ${y}-1 1 0 0 0</pose>
+                  <pose>1 -1 1 0 0 0</pose>
               </waypoint>
               <waypoint>
                   <time>4.0</time>
-                  <pose>${x}-1 ${y}-1 1 0 0 0</pose>
+                  <pose>-1 -1 1 0 0 0</pose>
               </waypoint>
             </trajectory>

File: usv_worlds/worlds/simple_obstacles.xacro (robot description, xacro)
@@ -5,17 +5,18 @@
   <xacro:include filename="$(find usv_worlds)/worlds/simple_box.xacro" />
   <xacro:macro name="simple_obstacles">
-    <xacro:simple_box name="box_north" x="100" y="60" Y="200" />
-    <xacro:simple_box name="box_south" x="-50" y="60" Y="200" />
+    <!--<xacro:simple_box name="box_north" x="100" y="60" Y="220" />
+    <xacro:simple_box name="box_south" x="-50" y="60" Y="220" />
     <xacro:simple_box name="box_east" x="25" y="-40" X="150" />
-    <xacro:simple_box name="box_west" x="-10" y="160" X="80" />
+    <xacro:simple_box name="box_west" x="25" y="160" X="150" /> -->
     <!--  Boxes to do static avoidance -->
-    <xacro:simple_box name="box_test" x="30" y="30" X="1" Y="1" Z="2" />
-    <xacro:simple_box name="box_test_two" x="15" y="15" X="2" Y="2" Z="2" />
-    <xacro:simple_box name="box_test_three" x="25" y="25" X="20" Y="20" Z="2" />
-    <xacro:simple_box name="box_test_four" x="23" y="20" X="20" Y="20" Z="2" />
+    <!--<xacro:simple_box name="box_test" x="30" y="30" X="2" Y="2" Z="2" />
+    <xacro:simple_box name="box_test2" x="25" y="30" X="2" Y="2" Z="2" />
+    <xacro:simple_box name="box_test3" x="22" y="30" X="2" Y="2" Z="2" />
+    <xacro:simple_box name="box_test4" x="15" y="30" X="2" Y="2" Z="2" />
+    <xacro:simple_box name="box_test5" x="35" y="30" X="2" Y="2" Z="2" />-->
+    <xacro:simple_box name="box_test" x="40" y="22" X="5" Y="5" Z="2" />
+    <xacro:simple_box name="box_test_two" x="20" y="8" X="3" Y="3" Z="2" />
+    <!--<xacro:simple_box name="box_test_three" x="25" y="25" X="2" Y="2" Z="2" />
+    <xacro:simple_box name="box_test_four" x="23" y="25" X="2" Y="2" Z="2" />-->
   </xacro:macro>
 </world>
-    <!--<xacro:simple_box name="jetty_one" x="-17.5" y="7" z="0.50" X="65" Y="3" Z="1.0" color="Wood" />
-    <xacro:simple_box name="jetty_two" x="-7.5" y="64" z="0.50" X="85" Y="4" Z="1.0" color="Wood" />
-    <xacro:simple_box name="jetty_three" x="92.5" y="74" z="0.50" X="5" Y="112" Z="1.0" color="Wood" />
-    <xacro:simple_box name="box_north2" x="10" y="-20" Y="100" yaw="-1.0" /> -->

File: usv_worlds/worlds/usv.world.xacro (robot description, xacro)
@@ -10,5 +10,5 @@
       </sky>
       <grid>false</grid>
-      <origin_visual>false</origin_visual>
+      <origin_visual>true</origin_visual>
     </scene>
     <!-- Estimated latitude/longitude of Trondheim harbor from satellite imagery -->
@@ -37,8 +37,12 @@
     <!-- Some simple obstacles in the way-->
     <!--<xacro:include filename="$(find usv_worlds)/worlds/simple_obstacles.xacro" />
-    <xacro:simple_obstacles /> -->
+    <xacro:simple_obstacles />-->
     <!-- simple trajectory to navigate between walls-->
     <xacro:include filename="$(find usv_worlds)/worlds/Obstacle_Path.xacro" />
     <xacro:Obstacle_Path />
+    <!-- First test with dynamic obstacle without changing anything -->
+    <!--<xacro:include filename="$(find usv_worlds)/worlds/moving_obstacles.xacro" />
+    <xacro:moving_obstacles /> -->
+     <!-- CUSTOM Ground Plane -->
   </world>
 </sdf>
